File: keyboard-pcb/keyboard-pcb.kicad_sch (KiCad schematic)
At the start: 131 parts

Commit message: assigned footprints and fixed naming
Parts:
- ALT1, ALT2, CAP1, CTRL1, FNC1, MX48, SHFT1, SUP1: renamed from MX?; footprint (none) -> Button_Switch_Keyboard:SW_Cherry_MX_1.25u_PCB
- BKSP1, TAB1: renamed from MX?; footprint (none) -> Button_Switch_Keyboard:SW_Cherry_MX_1.50u_PCB
- D1, D10, D11, D12, D13, D14, D15, D16, D17, D18, D19, D2, D20, D21, D22, D23, D24, D25, D26, D27, D28, D29, D3, D30, D31, D32, D33, D34, D35, D36, D37, D38, D39, D4, D40, D41, D42, D43, D44, D45, D46, D47, D48, D49, D5, D50, D51, D52, D53, D54, D55, D56, D57, D58, D59, D6, D60, D61, D62, D63, D64, D65, D7, D8, D9: renamed from D?; footprint (none) -> Diode_SMD:D_SOD-123
- DEL1, DWN1, LFT1, MX1, MX10, MX11, MX12, MX13, MX14, MX15, MX16, MX17, MX18, MX19, MX2, MX20, MX21, MX22, MX23, MX24, MX25, MX26, MX27, MX28, MX29, MX3, MX30, MX31, MX32, MX33, MX34, MX35, MX36, MX37, MX38, MX39, MX4, MX40, MX41, MX42, MX43, MX44, MX45, MX46, MX47, MX5, MX6, MX7, MX8, MX9, RHT1, UP1: renamed from MX?; footprint (none) -> Button_Switch_Keyboard:SW_Cherry_MX_1.00u_PCB
- ENT1: renamed from MX?; footprint (none) -> Button_Switch_Keyboard:SW_Cherry_MX_1.75u_PCB
- SPC1: renamed from MX?; footprint (none) -> Button_Switch_Keyboard:SW_Cherry_MX_6.25u_PCB
- SW1: renamed from SW?; footprint (none) -> Rotary_Encoder:RotaryEncoder_Alps_EC11E-Switch_Vertical_H20mm
- gave numbers to parts that had none: 1
