File: keyboard-pcb/keyboard-pcb.kicad_sch (KiCad schematic)
At the start: 131 parts, among them SW1 RotaryEncoder_Switch, U1 Pico

Commit message: added footprints to pcb editor
Parts:
- U1: footprint RPi_Pico:RPi_Pico_SMD_TH -> MCU_RaspberryPi_and_Boards:RPi_Pico_SMD_TH
Changed lines of the file:
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@@
     (property "Reference" "U1" (id 0) (at 76.2 36.83 0))
     (property "Value" "Pico" (id 1) (at 76.2 39.37 0))
-    (property "Footprint" "RPi_Pico:RPi_Pico_SMD_TH" (id 2) (at 76.2 68.58 90)
+    (property "Footprint" "MCU_RaspberryPi_and_Boards:RPi_Pico_SMD_TH" (id 2) (at 76.2 68.58 90)
       (effects (font (size 1.27 1.27)) hide)
     )
@@
     )
     (path "/f433be38-82e2-473b-9bcf-c0c050d04e9a"
-      (reference "U1") (unit 1) (value "Pico") (footprint "RPi_Pico:RPi_Pico_SMD_TH")
+      (reference "U1") (unit 1) (value "Pico") (footprint "MCU_RaspberryPi_and_Boards:RPi_Pico_SMD_TH")
     )
     (path "/c4b08a63-44b5-48b9-adfd-68736c92ed66"

Commit message: fixed error in schematic and moved rotary encoder up
Connections:
- net COL_13: now also RHT1.1 (COL), UP1.1 (COL)
- net ROW_1: now also D65.1 (K); no longer D62.1 (K)
- net ROW_2: now also D62.1 (K); no longer D65.1 (K), RHT1.1 (COL), UP1.1 (COL)
Other:
- moved on the sheet: D62, D65, DEL1, SW1

Commit message: added column GPIO tracks - pcb completed
Connections:
- net COL_0: now also U1.17 (GPIO13); no longer U1.20 (GPIO15)
- net COL_10: now also U1.6 (GPIO4); no longer U1.7 (GPIO5)
- net COL_11: now also U1.7 (GPIO5); no longer U1.6 (GPIO4)
- net COL_12: now also U1.9 (GPIO6); no longer U1.5 (GPIO3)
- net COL_13: now also U1.10 (GPIO7); no longer U1.4 (GPIO2)
- net COL_2: now also U1.20 (GPIO15); no longer U1.17 (GPIO13)
- net COL_8: now also U1.4 (GPIO2); no longer U1.10 (GPIO7)
- net COL_9: now also U1.5 (GPIO3); no longer U1.9 (GPIO6)

Commit message: corrected rotary encoder schematic + pcb
+ needed to be rotated
+ removed backups
Connections:
- net CLK: now also SW1.A; no longer SW1.S2
- net DT: now also SW1.B; no longer SW1.S1
- net GND: now also SW1.S2; no longer SW1.A
- net at D65.2 (A): now also SW1.S1; no longer SW1.B
Other:
- moved on the sheet: SW1
Changed lines of the file:
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@@
+    (stroke (width 0) (type default) (color 0 0 0 0))
+  )
+  (wire (pts (xy 323.85 162.56) (xy 358.14 162.56))
     (stroke (width 0) (type default) (color 0 0 0 0))
   )
@@
     (stroke (width 0) (type default) (color 0 0 0 0))
   )
-  (wire (pts (xy 326.39 154.94) (xy 330.2 154.94))
-    (stroke (width 0) (type default) (color 0 0 0 0))
-  )
   (wire (pts (xy 262.89 193.04) (xy 265.43 193.04))
     (stroke (width 0) (type default) (color 0 0 0 0))
@@
     (stroke (width 0) (type default) (color 0 0 0 0))
   )
+  (wire (pts (xy 326.39 154.94) (xy 345.44 154.94))
+    (stroke (width 0) (type default) (color 0 0 0 0))
+  )
   (wire (pts (xy 220.98 175.26) (xy 223.52 175.26))
     (stroke (width 0) (type default) (color 0 0 0 0))
@@
   )
   (wire (pts (xy 193.04 157.48) (xy 195.58 157.48))
-    (stroke (width 0) (type default) (color 0 0 0 0))
-  )
-  (wire (pts (xy 323.85 162.56) (xy 358.14 162.56))
     (stroke (width 0) (type default) (color 0 0 0 0))
   )
@@
     (pin "2")
   )
-  (symbol (lib_id "Device:RotaryEncoder_Switch") (at 337.82 154.94 0) (unit 1)
+  (symbol (lib_id "Device:RotaryEncoder_Switch") (at 337.82 154.94 180) (unit 1)
     (in_bom yes) (on_board yes) (fields_autoplaced)
     (property "Reference" "SW1" (id 0) (at 337.82 144.78 0))
     (property "Value" "RotaryEncoder_Switch" (id 1) (at 337.82 147.32 0))
-    (property "Footprint" "Rotary_Encoder:RotaryEncoder_Alps_EC11E-Switch_Vertical_H20mm" (id 2) (at 334.01 150.876 0)
-      (effects (font (size 1.27 1.27)) hide)
-    )
-    (property "Datasheet" "~" (id 3) (at 337.82 148.336 0)
-      (effects (font (size 1.27 1.27)) hide)
-    )
+    (property "Footprint" "Rotary_Encoder:RotaryEncoder_Alps_EC11E-Switch_Vertical_H20mm" (id 2) (at 341.63 159.004 0)
+      (effects (font (size 1.27 1.27)) hide)
+    )
+    (property "Datasheet" "~" (id 3) (at 337.82 161.544 0)
+      (effects (font (size 1.27 1.27)) hide)
+    )
