File: keyboard-pcb/keyboard-pcb.kicad_pcb (KiCad board)
At the start: 2 copper layers, 131 parts, among them SW1 RotaryEncoder_Switch, U1 Pico

Commit message: initial pcb layout
Parts:
- moved U1 271.0 mm to (358.0, 164.7)
- moved SHFT1 228.3 mm to (51.2, 177.8)
- moved MX3 228.1 mm to (77.4, 139.7)
- moved D62 223.6 mm to (295.3, 146.1), turned to 90 degrees
- moved D65 217.9 mm to (311.1, 132.1), turned to 90 degrees
- moved DWN1 213.1 mm to (306.0, 196.9)
- moved MX6 211.7 mm to (86.9, 120.7)
- moved MX11 205.6 mm to (115.5, 139.7)
- moved BKSP1 204.0 mm to (301.2, 120.7)
- moved MX24 199.3 mm to (177.4, 158.8)
- moved SW1 191.6 mm to (315.0, 123.2)
- moved D60 189.5 mm to (295.3, 203.2), turned to 90 degrees
- moved MX1 189.3 mm to (48.8, 120.7)
- moved D63 186.1 mm to (295.3, 184.2), turned to 90 degrees
- moved MX21 182.4 mm to (148.8, 177.8)
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
Commit message: diodes and mcu flipped to other side of board
Parts:
- D1, D10, D11, D12, D13, D14, D15, D16, D17, D18, D19, D2, D20, D21, D22, D23, D24, D25, D26, D27, D28, D29, D3, D30, D31, D32, D33, D34, D35, D36, D37, D38, D39, D4, D40, D41, D42, D43, D44, D45, D46, D47, D48, D49, D5, D50, D51, D52, D53, D54, D55, D56, D57, D58, D59, D6, D60, D61, D62, D63, D64, D65, D7, D8, D9, U1: moved to B.Cu
- turned U1 to 180 degrees

Commit message: no changes
Parts:
- moved ALT2 30.4 mm to (268.5, 182.4)
- moved D42 30.4 mm to (245.8, 131.6)
- moved MX29 30.4 mm to (213.7, 163.3)
- moved D12 30.4 mm to (112.4, 131.6)
- moved D21 30.4 mm to (150.5, 131.6)
- moved D27 30.4 mm to (164.9, 169.7)
- moved D33 30.4 mm to (198.2, 112.5)
- moved MX19 30.4 mm to (180.3, 125.2)
- moved MX36 30.4 mm to (261.3, 144.3)
- moved SPC1 30.4 mm to (197.0, 182.4)
- moved MX6 30.4 mm to (113.7, 106.2)
- moved CTRL1 30.4 mm to (78.0, 182.4)
- moved ALT1 30.4 mm to (125.6, 182.4)
- moved D17 30.4 mm to (131.5, 131.6)
- moved D2 30.4 mm to (68.6, 131.6)
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
Commit message: added edge cuts
Parts:
- moved D60 5.38 mm to (327.1, 190.5)
- moved D62 5.38 mm to (327.1, 133.3)
- moved D64 5.38 mm to (346.1, 190.5)
- moved MX48 5.38 mm to (316.4, 165.1)
- moved MX35 5.38 mm to (261.6, 127.0)
- moved MX39 5.38 mm to (280.6, 127.0)
- moved SW1 5.38 mm to (346.8, 110.5)
- moved D49 5.38 mm to (265.2, 171.4)
- moved D51 5.38 mm to (279.5, 114.3)
- moved D56 5.38 mm to (298.5, 114.3)
- moved D58 5.38 mm to (318.8, 152.4)
- moved D63 5.38 mm to (327.1, 171.4)
- moved D65 5.38 mm to (343.0, 119.4)
- moved MX40 5.38 mm to (285.4, 146.0)
- moved MX44 5.38 mm to (304.5, 146.0)
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Other:
- board outline added: 303.5 x 96.5 mm

Commit message: fixed edge cut where it was going through holes
Other:
- board size 303.5 x 96.5 mm -> 303.5 x 97.8 mm
Changed lines of the file:
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@@
   )
   (gr_arc (start 369.57 102.87) (mid 370.468026 103.241974) (end 370.84 104.14) (layer "Edge.Cuts") (width 0.2))
-  (gr_line (start 369.57 199.39) (end 68.58 199.39) (layer "Edge.Cuts") (width 0.2))
-  (gr_line (start 67.31 198.12) (end 67.31 104.14) (layer "Edge.Cuts") (width 0.2))
-  (gr_arc (start 370.84 198.12) (mid 370.468026 199.018026) (end 369.57 199.39) (layer "Edge.Cuts") (width 0.2))
+  (gr_line (start 369.57 200.66) (end 68.58 200.66) (layer "Edge.Cuts") (width 0.2))
+  (gr_line (start 67.31 199.39) (end 67.31 104.14) (layer "Edge.Cuts") (width 0.2))
+  (gr_arc (start 68.58 200.66) (mid 67.681974 200.288026) (end 67.31 199.39) (layer "Edge.Cuts") (width 0.2))
   (gr_arc (start 67.31 104.14) (mid 67.681974 103.241974) (end 68.58 102.87) (layer "Edge.Cuts") (width 0.2))
-  (gr_line (start 370.84 104.14) (end 370.84 198.12) (layer "Edge.Cuts") (width 0.2))
-  (gr_arc (start 68.58 199.39) (mid 67.681974 199.018026) (end 67.31 198.12) (layer "Edge.Cuts") (width 0.2))
+  (gr_line (start 370.84 104.14) (end 370.84 199.39) (layer "Edge.Cuts") (width 0.2))
+  (gr_arc (start 370.84 199.39) (mid 370.468026 200.288026) (end 369.57 200.66) (layer "Edge.Cuts") (width 0.2))
   (gr_line (start 68.58 102.87) (end 369.57 102.87) (layer "Edge.Cuts") (width 0.2))
 )

Commit message: routed key matric with tracks
+ rows and rotary encoder connected to GPIO pins
* still need to connect remaining columns
Parts:
- moved D58 2.59 mm to (316.2, 152.4)
- moved D65 2.08 mm to (340.9, 119.4)
Connections:
- D62 pad 1: ROW_1 -> ROW_2
- D65 pad 1: ROW_2 -> ROW_1
- RHT1 pad 1: ROW_2 -> COL_13
- UP1 pad 1: ROW_2 -> COL_13
Routing:
- net ROW_1: track 0.00 -> 321.4 mm
- net ROW_0: track 0.00 -> 320.7 mm
- net ROW_2: track 0.00 -> 315.8 mm
- net ROW_4: track 0.00 -> 299.7 mm
- net ROW_3: track 0.00 -> 276.9 mm
- net COL_13: track 0.00 -> 137.7 mm
- net COL_12: track 0.00 -> 117.4 mm
- net COL_11: track 0.00 -> 108.8 mm
- net COL_10: track 0.00 -> 107.5 mm
- net COL_9: track 0.00 -> 102.9 mm
- net COL_2: track 0.00 -> 93.0 mm
- net COL_1: track 0.00 -> 90.1 mm
- net COL_6: track 0.00 -> 89.8 mm
- net COL_0: track 0.00 -> 81.5 mm
- net COL_8: track 0.00 -> 70.0 mm
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
Commit message: fixed track on pcb
Routing:
- net ROW_0: track 320.7 -> 318.5 mm
Changed lines of the file:
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@@
   (segment (start 73.3218 186.69) (end 71.1708 188.841) (width 0.25) (layer "B.Cu") (net 9))
   (segment (start 76.6826 186.69) (end 73.3218 186.69) (width 0.25) (layer "B.Cu") (net 9))
+  (segment (start 342.646 119.38) (end 335.534 119.38) (width 0.25) (layer "B.Cu") (net 10))
   (segment (start 343.154 159.512) (end 343.653 160.011) (width 0.25) (layer "B.Cu") (net 10))
-  (segment (start 321.3608 115.941) (end 343.017 115.941) (width 0.25) (layer "B.Cu") (net 10))
+  (segment (start 335.534 119.38) (end 332.095 115.941) (width 0.25) (layer "B.Cu") (net 10))
+  (segment (start 332.095 115.941) (end 321.3608 115.941) (width 0.25) (layer "B.Cu") (net 10))
   (segment (start 69.9008 115.941) (end 321.3608 115.941) (width 0.25) (layer "B.Cu") (net 10))
-  (segment (start 343.154 116.078) (end 343.154 159.512) (width 0.25) (layer "B.Cu") (net 10))
+  (segment (start 343.154 119.888) (end 342.646 119.38) (width 0.25) (layer "B.Cu") (net 10))
+  (segment (start 343.154 159.512) (end 343.154 119.888) (width 0.25) (layer "B.Cu") (net 10))
   (segment (start 343.653 160.011) (end 346.8878 160.011) (width 0.25) (layer "B.Cu") (net 10))
-  (segment (start 343.017 115.941) (end 343.154 116.078) (width 0.25) (layer "B.Cu") (net 10))
   (segment (start 74.295 110.49) (end 72.0518 110.49) (width 0.25) (layer "B.Cu") (net 11))
   (segment (start 72.0518 110.49) (end 69.9008 112.641) (width 0.25) (layer "B.Cu") (net 11))
@@
   (segment (start 348.2768 186.69) (end 346.1258 188.841) (width 0.25) (layer "B.Cu") (net 73))
   (segment (start 350.52 186.69) (end 348.2768 186.69) (width 0.25) (layer "B.Cu") (net 73))
-  (segment (start 344.745 117.602) (end 340.868 117.602) (width 0.25) (layer "F.Cu") (net 74))
-  (segment (start 346.826 115.521) (end 344.745 117.602) (width 0.25) (layer "F.Cu") (net 74))
+  (segment (start 343.068 115.521) (end 340.868 117.721) (width 0.25) (layer "B.Cu") (net 74))
+  (segment (start 346.826 115.521) (end 343.068 115.521) (width 0.25) (layer "B.Cu") (net 74))
   (segment (start 319.786 130.81) (end 319.786 142.24) (width 0.25) (layer "F.Cu") (net 75))
   (segment (start 318.7446 126.991) (end 318.7446 129.7686) (width 0.25) (layer "F.Cu") (net 75))

Commit message: added column GPIO tracks - pcb completed
Connections:
- U1 pad 10: COL_8 -> COL_13
- U1 pad 17: COL_2 -> COL_0
- U1 pad 20: COL_0 -> COL_2
- U1 pad 4: COL_13 -> COL_8
- U1 pad 5: COL_12 -> COL_9
- U1 pad 6: COL_11 -> COL_10
- U1 pad 7: COL_10 -> COL_11
- U1 pad 9: COL_9 -> COL_12
Routing:
- net COL_0: track 81.5 -> 402.2 mm
- net COL_1: track 90.1 -> 380.7 mm
- net COL_3: track 69.7 -> 345.3 mm
- net COL_2: track 93.0 -> 355.7 mm
- net COL_4: track 69.6 -> 328.7 mm
- net COL_5: track 69.8 -> 313.0 mm
- net COL_7: track 69.8 -> 279.3 mm
- net COL_6: track 89.8 -> 295.6 mm
- net COL_8: track 70.0 -> 223.1 mm
- net COL_9: track 102.9 -> 237.5 mm
- net COL_10: track 107.5 -> 229.4 mm
- net COL_11: track 108.8 -> 213.9 mm
- net COL_12: track 117.4 -> 208.2 mm
- net COL_13: track 137.7 -> 153.7 mm
