File: keyboard-pcb/keyboard-pcb.kicad_pcb (KiCad board)
At the start: 2 copper layers, 303.5 x 97.8 mm, 131 parts, among them SW1 RotaryEncoder_Switch, U1 Pico

Commit message: DRC and Parity check run
+ corrected errors fixing - silkscreens and unconnected wires
Parts:
- moved D18 0.43 mm to (140.8, 152.4)
- moved D22 0.43 mm to (159.9, 152.4)
- moved D30 0.43 mm to (198.0, 152.4)
- moved D39 0.43 mm to (236.1, 152.4)
- moved D43 0.43 mm to (255.1, 152.4)
- moved D48 0.43 mm to (274.2, 152.4)
- moved D53 0.43 mm to (293.2, 152.4)
- moved D8 0.43 mm to (102.7, 152.4)
- moved D1 0.43 mm to (69.5, 114.3)
- moved D24 0.43 mm to (164.7, 114.3)
- moved D33 0.43 mm to (202.8, 114.3)
- moved D37 0.43 mm to (221.9, 114.3)
- moved D46 0.43 mm to (260.0, 114.3)
- moved D51 0.43 mm to (279.0, 114.3)
- moved D56 0.43 mm to (298.1, 114.3)
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Routing:
- net COL_8: track 223.1 -> 222.1 mm

Commit message: pcb modifications
+ added footprint cutout for RP Pico so pads on RP Pico can be accessed
+ rerouted some tracks and cleaned up
+ DRC checked with parity
Routing:
- net COL_10: track 229.4 -> 233.2 mm
- net COL_11: track 213.9 -> 215.1 mm

Commit message: silkscreen name added and gerbers generated
Other:
- board text added: "Orions Hands"
- board text added: "V1.0"
Changed lines of the file:
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@@
   (gr_arc (start 370.84 199.39) (mid 370.468026 200.288026) (end 369.57 200.66) (layer "Edge.Cuts") (width 0.2))
   (gr_line (start 68.58 102.87) (end 369.57 102.87) (layer "Edge.Cuts") (width 0.2))
+  (gr_text "V1.0" (at 178.308 189.484) (layer "F.SilkS")
+    (effects (font (size 1.5 3) (thickness 0.3) italic))
+  )
+  (gr_text "Orions Hands" (at 229.362 189.738) (layer "F.SilkS")
+    (effects (font (size 1.5 3) (thickness 0.3) italic))
+  )
   (segment (start 118.745 110.363) (end 119.634 111.252) (width 0.25) (layer "F.Cu") (net 1))
   (segment (start 123.4948 167.4368) (end 124.46 168.402) (width 0.25) (layer "F.Cu") (net 1))
