File: keyboard-pcb/keyboard-pcb.kicad_pcb (KiCad board)
At the start: 2 copper layers, 303.5 x 97.8 mm, 131 parts, among them SW1 RotaryEncoder_Switch, U1 Pico

Commit message: updated pcb with silkscreen and new gerber files
+ silkscreen required for printing with jlcpcb
Other:
- board text added: "JLCJLCJLCJLC"
Changed lines of the file:
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@@
   (gr_arc (start 370.84 199.39) (mid 370.468026 200.288026) (end 369.57 200.66) (layer "Edge.Cuts") (width 0.2))
   (gr_line (start 68.58 102.87) (end 369.57 102.87) (layer "Edge.Cuts") (width 0.2))
+  (gr_text "JLCJLCJLCJLC" (at 355.6 160.02 90) (layer "B.SilkS")
+    (effects (font (size 0.8 0.8) (thickness 0.15)) (justify mirror))
+  )
   (gr_text "V1.0" (at 178.308 189.484) (layer "F.SilkS")
     (effects (font (size 1.5 3) (thickness 0.3) italic))

Commit message: corrected rotary encoder schematic + pcb
+ needed to be rotated
+ removed backups
Parts:
- moved SW1 7.68 mm to (354.1, 113.0), turned to 180 degrees
Connections:
- SW1 pad A: GND -> CLK
- SW1 pad B: Net-(D65-Pad2) -> DT
- SW1 pad S1: DT -> Net-(D65-Pad2)
- SW1 pad S2: CLK -> GND
Routing:
- net COL_13: track 153.7 -> 195.2 mm
- net DT: track 13.7 -> 21.8 mm
- net CLK: track 15.3 -> 10.2 mm
- net Net-(D65-Pad2): track 6.87 -> 9.76 mm
- net GND: track 32.1 -> 29.9 mm

Commit message: corrected version + cleaned up images
+ adding images to separate folder
Other:
- board text added: "V0.1"
- board text removed: "V1.0"
Changed lines of the file:
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@@
     (effects (font (size 0.8 0.8) (thickness 0.15)) (justify mirror))
   )
-  (gr_text "V1.0" (at 178.308 189.484) (layer "F.SilkS")
+  (gr_text "V0.1" (at 178.308 189.484) (layer "F.SilkS")
     (effects (font (size 1.5 3) (thickness 0.3) italic))
   )
