File: keyboard-pcb/keyboard-pcb_firmware_version.kicad_pcb (KiCad board)
At the start: 2 copper layers, 303.5 x 97.8 mm, 131 parts, among them SW1 RotaryEncoder_Switch, U1 Pico

Commit message: corrected version + cleaned up images
+ adding images to separate folder
Other:
- board text added: "V0.1"
- board text removed: "V1.0"
Changed lines of the file:
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@@
     (property "Sheetname" "")
     (attr smd)
-    (fp_text reference "D1" (at 0 2 90) (layer "B.SilkS")
+    (fp_text reference "D1" (at 3.5052 -0.0254 90) (layer "B.SilkS")
       (effects (font (size 1 1) (thickness 0.15)) (justify mirror))
     )
@@
     (effects (font (size 0.8 0.8) (thickness 0.15)) (justify mirror))
   )
-  (gr_text "V1.0" (at 178.308 189.484) (layer "F.SilkS")
+  (gr_text "V0.1" (at 178.308 189.484) (layer "F.SilkS")
     (effects (font (size 1.5 3) (thickness 0.3) italic))
   )
